Commit message: feat(uika): update robot model geometry

File: source/himloco_lab/himloco_lab/assets/uika/urdf/uika.urdf (robot description, URDF)
Before this commit: robot UIKA, 17 links, 16 joints
Links:
- link base: mass 6.09961854 -> 6.47472235
Joints:
- joint FL_calf_joint: axis 0 0.716968137917877 0.69710593829817 -> 0 0.753262811155552 0.657719649493639; origin xyz=-0.152475747348646 0.109582492974347 -0.07397319848129 rpy=0 0 0 -> xyz=-0.152226491053868 0.105657558324466 -0.0799549009122722 rpy=0 0 0
- joint FL_foot_joint: origin xyz=0.211725899509592 -0.00252783551179853 -0.0167659233263265 rpy=0 0 0 -> xyz=0.211745241606516 -0.00368975133737329 -0.016299725536693 rpy=0 0 0
- joint FL_thigh_joint: axis 0 0.716968137917879 0.697105938298167 -> 0 0.753262811155553 0.657719649493638; origin xyz=0.0560002942624635 0.0483946520428511 0.0470555828957988 rpy=0 0 0 -> xyz=0.0560002933981102 0.0508445597819099 0.0443970251456514 rpy=0 0 0
- joint FR_calf_joint: axis 0 0.716968137917903 -0.697105938298144 -> 0 0.753262811155038 -0.657719649494228; origin xyz=-0.152475581141278 -0.109581813299707 -0.0739724994411187 rpy=0 0 0 -> xyz=-0.152226326722374 -0.105656916842211 -0.079954166245416 rpy=0 0 0
- joint FR_foot_joint: origin xyz=0.211725899509592 0.00252783231169756 -0.0167659202148746 rpy=0 0 0 -> xyz=0.211745241606515 0.00368974797525654 -0.0162997226010469 rpy=0 0 0
- joint FR_thigh_joint: axis 0 0.716968137917902 -0.697105938298144 -> 0 0.753262811155038 -0.657719649494228; origin xyz=0.0560001425520644 -0.0483952686957443 0.047054585042635 rpy=0 0 0 -> xyz=0.0560001435635803 -0.0508451382424889 0.0443959916658049 rpy=0 0 0
- joint RL_calf_joint: axis 0 0.716968137917874 0.697105938298173 -> 0 0.753262811155552 0.657719649493639; origin xyz=-0.152475747348643 0.109582492974347 -0.0739731984812923 rpy=0 0 0 -> xyz=-0.152226491053865 0.105657558324469 -0.0799549009122762 rpy=0 0 0
- joint RL_foot_joint: origin xyz=0.211725899509589 -0.00252783551179986 -0.0167659233263231 rpy=0 0 0 -> xyz=0.211745241606513 -0.00368975133737642 -0.0162997255366898 rpy=0 0 0
- joint RL_thigh_joint: axis 0 0.716968137917878 0.697105938298169 -> 0 0.753262811155552 0.657719649493639; origin xyz=-0.0559996912405691 0.0483949903212994 0.0470544297768458 rpy=0 0 0 -> xyz=-0.0559996921049242 0.0508448980603474 0.044395872026712 rpy=0 0 0
- joint RR_calf_joint: axis 0 0.716968137917903 -0.697105938298143 -> 0 0.753262811155037 -0.657719649494229; origin xyz=-0.152475581141278 -0.109581813299707 -0.0739724994411164 rpy=0 0 0 -> xyz=-0.152226326722374 -0.105656916842211 -0.079954166245416 rpy=0 0 0
- joint RR_foot_joint: origin xyz=0.211725899509593 0.00252783231169423 -0.0167659202148782 rpy=0 0 0 -> xyz=0.211745241606515 0.00368974797525667 -0.0162997226010466 rpy=0 0 0
- joint RR_thigh_joint: axis 0 0.716968137917902 -0.697105938298144 -> 0 0.753262811155037 -0.657719649494228; origin xyz=-0.0559998574479382 -0.0483962427296829 0.0470544132941808 rpy=0 0 0 -> xyz=-0.0559998564364221 -0.0508461122763563 0.0443958199174349 rpy=0 0 0
